File: corne-chocolate/pcb/corne-chocolate.kicad_pcb (KiCad board)
At the start: 2 copper layers, 133.8 x 91.4 mm, 98 parts, among them J3 LED, P1 i2c-pin, P2 i2c-pin, SW1 SW_PUSH, SW10 SW_PUSH, SW11 SW_PUSH, SW12 SW_PUSH, SW13 SW_PUSH, SW14 SW_PUSH, SW15 SW_PUSH, SW16 SW_PUSH, SW17 SW_PUSH, SW18 SW_PUSH, SW19 SW_PUSH, SW2 SW_PUSH, SW20 SW_PUSH, SW21 SW_PUSH, SW3 SW_PUSH, SW4 SW_PUSH, SW5 SW_PUSH, SW6 SW_PUSH, SW7 SW_PUSH, SW8 SW_PUSH, SW9 SW_PUSH, U1 ProMicro

Commit message: add new stuff
Parts:
- added D22: D, kbd:D3_TH_SMD, F.Cu at (171.4, 137.4)
- added L28: SK6812MINI, kbd:SK6812MINI_rev, F.Cu at (176.9, 138.7)
- added SW22: SW_PUSH, kbd:MX_ALPS_PG1350_noLed, F.Cu at (181.4, 141.3)
- added SW23: Rotary_Encoder, Rotary_Encoder:RotaryEncoder_Alps_EC11E_Vertical_H20mm, F.Cu at (214.3, 120.3)
- D1, D10, D11, D12, D13, D14, D15, D16, D17, D18, D19, D2, D20, D21, D3, D4, D5, D6, D7, D8, D9: footprint kbd:D3_SMD -> kbd:D3_TH_SMD
- RSW1: value Reset -> SW_PUSH
- SW1, SW10, SW11, SW12, SW13, SW14, SW15, SW16, SW17, SW18, SW19, SW2, SW20, SW3, SW4, SW5, SW6, SW7, SW8, SW9: footprint kbd:Choc_Hotswap -> kbd:MX_ALPS_PG1350_noLed
- SW21: footprint kbd:Choc_Hotswap_1.5u -> kbd:MX_ALPS_PG1350_noLed_1.75u
- moved L21 21.4 mm to (191.8, 147.1)
- moved SW21 21.3 mm to (196.2, 150.0)
- moved D21 20.9 mm to (167.7, 133.1)
- moved ? 11.2 mm to (166.1, 141.2)
- moved ? 7.47 mm to (191.2, 131.7)
- moved ? 2.81 mm to (123.0, 125.5)
- renumbered TRRS to J1, OLED to J2, data to JP1
Connections:
- L15 pad 1: Net-(L14-Pad3) -> Net-(L15-Pad1)
Routing:
- net Net-(L15-Pad1): track 0.00 -> 106.2 mm, vias 0 -> 1
- net VCC: track 786.4 -> 752.2 mm, vias 30 -> 29
- net col5: track 188.2 -> 211.2 mm, vias 10 -> 9
- net GND: track 816.7 -> 839.7 mm, vias 59 -> 56
- net Net-(L18-Pad3): track 39.1 -> 59.1 mm, vias 6 -> 5
- net Net-(D22-Pad2): track 0.00 -> 19.8 mm
- net Net-(L21-Pad3): track 30.7 -> 14.6 mm, vias 4 -> 3
- net row3: track 119.2 -> 129.4 mm, vias 6 -> 5
- net row2: track 209.9 -> 204.6 mm, vias 15 -> 14
- net Net-(D21-Pad2): track 50.2 -> 46.7 mm, vias 2 -> 0
- net col3: track 224.8 -> 228.1 mm, vias 12 -> 11
- net Net-(D20-Pad2): track 25.8 -> 28.7 mm
- net Net-(D19-Pad2): track 21.2 -> 19.1 mm, vias 2 -> 1
- net col4: track 196.2 -> 195.0 mm, vias 8 -> 7
- removed copper zone on B.Cu, net GND
- removed copper zone on F.Cu, net GND
Other:
- board size 133.8 x 91.4 mm -> 149.8 x 119.3 mm
