File: corne-chocolate/pcb/corne-chocolate.sch (KiCad schematic (older format))
At the start: 87 parts, among them J1 MJ-4PP-9, J2 OLED, J3 LED, P1 i2c-pin, P2 i2c-pin, SW1 SW_PUSH, SW10 SW_PUSH, SW11 SW_PUSH, SW12 SW_PUSH, SW13 SW_PUSH, SW14 SW_PUSH, SW15 SW_PUSH, SW16 SW_PUSH, SW17 SW_PUSH, SW18 SW_PUSH, SW19 SW_PUSH, SW2 SW_PUSH, SW20 SW_PUSH, SW21 SW_PUSH, SW3 SW_PUSH, SW4 SW_PUSH, SW5 SW_PUSH, SW6 SW_PUSH, SW7 SW_PUSH, SW8 SW_PUSH, SW9 SW_PUSH, U1 ProMicro

Commit message: add new stuff
Parts:
- added D22: D, kbd:D3_TH_SMD, symbol Device:D
- added L28: SK6812MINI, kbd:SK6812MINI_rev, symbol corne-chocolate-rescue:SK6812MINI-kbd
- added SW22: SW_PUSH, kbd:keyswitch_cherrymx_alps_choc12_1.5u, symbol corne-chocolate-rescue:SW_PUSH-kbd
- added SW23: Rotary_Encoder, Rotary_Encoder:RotaryEncoder_Alps_EC11E_Vertical_H20mm, symbol Device:Rotary_Encoder
- J1: symbol kbd:MJ-4PP-9 -> corne-chocolate-rescue:MJ-4PP-9-kbd
- L1, L10, L11, L12, L13, L14, L15, L16, L17, L18, L19, L2, L20, L21, L3, L4, L5, L6, L7, L8, L9: symbol kbd:SK6812MINI -> corne-chocolate-rescue:SK6812MINI-kbd
- L22, L23, L24, L25, L26, L27: footprint kbd:SK6812MINI_underglow -> kbd:SK6812MINI_underglow_rev; symbol kbd:SK6812MINI -> corne-chocolate-rescue:SK6812MINI-kbd
- RSW1: symbol kbd:SW_PUSH -> corne-chocolate-rescue:SW_PUSH-kbd
- SW1, SW10, SW11, SW12, SW13, SW14, SW15, SW16, SW17, SW18, SW19, SW2, SW20, SW3, SW4, SW5, SW6, SW7, SW8, SW9: footprint kbd:MX_ALPS_PG1350_noLed -> kbd:keyswitch_cherrymx_alps_choc12_1u; symbol kbd:SW_PUSH -> corne-chocolate-rescue:SW_PUSH-kbd
- SW21: footprint kbd:MX_ALPS_PG1350_noLed_1.75u -> kbd:keyswitch_cherrymx_alps_choc12_1.5u; symbol kbd:SW_PUSH -> corne-chocolate-rescue:SW_PUSH-kbd
- U1: symbol kbd:ProMicro -> corne-chocolate-rescue:ProMicro-kbd
Connections:
- net labels added: ENCA, ENCB
- wire segments 265 -> 276
- no-connect marks 6 -> 4
